Commit message: fix robot model and add turret

File: explorer_bot/urdf/explorer_robot.urdf (robot description, URDF)
Before this commit: robot explorer_robot, 2 links, 1 joints
Links:
- removed link second_link
- added link base_footprint
- added link caster_wheel_link; visual sphere radius=0.06
- added link left_wheel_link; visual cylinder length=0.05 radius=0.1
- added link right_wheel_link; visual cylinder length=0.05 radius=0.1
- added link turret_bottom_link; visual cylinder length=0.05 radius=0.06
- added link turret_link; visual cylinder length=0.2 radius=0.05
- added link turret_top_link; visual cylinder length=0.05 radius=0.06
- link base_link: geometry visual cylinder length=0.14 radius=0.2
Joints:
- removed joint base_second_joint
- added joint base_caster_wheel_joint: type fixed, parent base_link, child caster_wheel_link, origin xyz=0.1 0 -0.05 rpy=0 0 0
- added joint base_joint: type fixed, parent base_footprint, child base_link, origin xyz=0 0 0.1 rpy=0 0 0
- added joint base_left_wheel_joint: type continuous, parent base_link, child left_wheel_link, origin xyz=-0.15 0.225 0 rpy=0 0 0, axis 0 1 0
- added joint base_right_wheel_joint: type continuous, parent base_link, child right_wheel_link, origin xyz=-0.15 -0.225 0 rpy=0 0 0, axis 0 1 0
- added joint base_turret_joint: type fixed, parent base_link, child turret_link, origin xyz=0 0 0.14 rpy=0 0 0
- added joint turret_bottom_joint: type fixed, parent turret_link, child turret_bottom_link, origin xyz=0 0 -0.075 rpy=0 0 0
- added joint turret_top_joint: type fixed, parent turret_link, child turret_top_link, origin xyz=0 0 0.175 rpy=0 0 0
