Commit message: add xacro to urdf

File: explorer_bot/urdf/explorer_robot.urdf.xacro (robot description, xacro)
@@ -1,4 +1,4 @@
 <?xml version="1.0"?>
-<robot name="explorer_robot">
+<robot name="explorer_robot" xmlns:xacro="http://www.ros.org/wiki/xacro">
     <material name="black">
         <color rgba="0 0 0 1" />
@@ -25,5 +25,5 @@
                 <cylinder radius="0.1" length="0.05" />
             </geometry>
-            <origin xyz="0.15 0 0" rpy="1.57 0 0" />
+            <origin xyz="0.15 0 0" rpy="${pi / 2.0} 0 0" />
             <material name="grey" />
         </visual>
@@ -34,5 +34,5 @@
                 <cylinder radius="0.1" length="0.05" />
             </geometry>
-            <origin xyz="0.15 0 0" rpy="1.57 0 0" />
+            <origin xyz="0.15 0 0" rpy="${pi / 2.0} 0 0" />
             <material name="grey" />
         </visual>

Commit message: add rviz config

File: explorer_bot/urdf/explorer_robot.urdf.xacro (robot description, xacro)
@@ -14,9 +14,20 @@
         <visual>
             <geometry>
-               <cylinder radius="0.2" length="0.14"/>
+                <cylinder radius="0.2" length="0.14"/>
             </geometry>
             <origin xyz="0 0 0.07" rpy="0 0 0" />
             <material name="black" />
         </visual>
+        <inertia>
+            <origin xyz="0 0 0.07" rpy="0 0 0" />
+            <mass value="1.0" />
+            <inertia ixx="0.001" ixy="0.0" ixz="0.0" iyy="0.001" iyz="0.0" izz="0.001" />
+        </inertia>
+        <collision>
+            <geometry>
+                <cylinder radius="0.2" length="0.14"/>
+            </geometry>
+            <origin xyz="0 0 0.07" rpy="0 0 0" />
+        </collision>
     </link>
     <link name="right_wheel_link">
@@ -28,4 +39,15 @@
             <material name="grey" />
         </visual>
+        <inertia>
+            <origin xyz="0.15 0 0" rpy="${pi / 2.0} 0 0" />
+            <mass value="0.5" />
+            <inertia ixx="0.0005" ixy="0.0" ixz="0.0" iyy="0.0005" iyz="0.0" izz="0.0005" />
+        </inertia>
+        <collision>
+            <geometry>
+                <cylinder radius="0.1" length="0.05"/>
+            </geometry>
+            <origin xyz="0.15 0 0" rpy="${pi / 2.0} 0 0" />
+        </collision>
     </link>
     <link name="left_wheel_link">
@@ -37,4 +59,15 @@
             <material name="grey" />
         </visual>
+        <inertia>
+            <origin xyz="0.15 0 0" rpy="${pi / 2.0} 0 0" />
+            <mass value="0.5" />
+            <inertia ixx="0.0005" ixy="0.0" ixz="0.0" iyy="0.0005" iyz="0.0" izz="0.0005" />
+        </inertia>
+        <collision>
+            <geometry>
+                <cylinder radius="0.1" length="0.05"/>
+            </geometry>
+            <origin xyz="0.15 0 0" rpy="${pi / 2.0} 0 0" />
+        </collision>
     </link>
     <link name="caster_wheel_link">
@@ -46,4 +79,15 @@
             <material name="grey" />
         </visual>
+        <inertia>
+            <origin xyz="0 0 0" rpy="0 0 0" />
+            <mass value="0.2" />
+            <inertia ixx="0.0001" ixy="0.0" ixz="0.0" iyy="0.0001" iyz="0.0" izz="0.0001" />
+        </inertia>
+        <collision>
+            <geometry>
+                <sphere radius="0.06"/>
+            </geometry>
+            <origin xyz="0 0 0" rpy="0 0 0" />
+        </collision>
     </link>
     <link name="turret_link">
@@ -55,4 +99,15 @@
             <material name="white"/>
         </visual>
+        <inertia>
+            <origin xyz="0 0 0.1" rpy="0 0 0" />
+            <mass value="0.3" />
+            <inertia ixx="0.0001" ixy="0.0" ixz="0.0" iyy="0.0001" iyz="0.0" izz="0.0001" />
+        </inertia>
+        <collision>
+            <geometry>
+                <cylinder radius="0.05" length="0.2"/>
+            </geometry>
+            <origin xyz="0 0 0.1" rpy="0 0 0" />
+        </collision>
     </link>
     <link name="turret_bottom_link">
@@ -64,4 +119,15 @@
             <material name="black"/>
         </visual>
+        <inertia>
+            <origin xyz="0 0 0.1" rpy="0 0 0" />
+            <mass value="0.2" />
+            <inertia ixx="0.00005" ixy="0.0" ixz="0.0" iyy="0.00005" iyz="0.0" izz="0.00005" />
+        </inertia>
+        <collision>
+            <geometry>
+                <cylinder radius="0.06" length="0.05"/>
+            </geometry>
+            <origin xyz="0 0 0.1" rpy="0 0 0" />
+        </collision>
     </link>
     <link name="turret_top_link">
@@ -73,4 +139,15 @@
             <material name="black"/>
         </visual>
+        <inertia>
+            <origin xyz="0 0 0.05" rpy="0 0 0" />
+            <mass value="0.2" />
+            <inertia ixx="0.00005" ixy="0.0" ixz="0.0" iyy="0.00005" iyz="0.0" izz="0.00005" />
+        </inertia>
+        <collision>
+            <geometry>
+                <cylinder radius="0.06" length="0.05"/>
+            </geometry>
+            <origin xyz="0 0 0.05" rpy="0 0 0" />
+        </collision>
     </link>
     <joint name="base_joint" type="fixed">

Commit message: replace bottom turret to lidar

File: explorer_bot/urdf/explorer_robot.urdf.xacro (robot description, xacro)
@@ -9,4 +9,7 @@
     <material name="grey">
         <color rgba="0.5 0.5 0.5 1" />
+    </material>
+    <material name="red">
+        <color rgba="1 0 0 1" />
     </material>
     <link name="base_footprint" />
@@ -111,5 +114,5 @@
         </collision>
     </link>
-    <link name="turret_bottom_link">
+    <link name="lidar_sensor">
         <visual>
             <geometry>
@@ -117,5 +120,5 @@
             </geometry>
             <origin xyz="0 0 0.1" rpy="0 0 0"/>
-            <material name="black"/>
+            <material name="red"/>
         </visual>
         <inertia>
@@ -180,5 +183,5 @@
     <joint name="turret_bottom_joint" type="fixed">
         <parent link="turret_link"/>
-        <child link="turret_bottom_link"/>
+        <child link="lidar_sensor"/>
         <origin xyz="0 0 -0.075" rpy="0 0 0"/>
     </joint>
