Commit message: fix robot physics

File: src/explorer_bot/urdf/mobile_base.xacro (robot description, xacro)
@@ -2,5 +2,5 @@
 <robot xmlns:xacro="http://www.ros.org/wiki/xacro">
     <xacro:property name="base_diameter" value="0.4" />
-    <xacro:property name="base_length" value="0.15" /> <!-- Length - wysokosc podstawy -->
+    <xacro:property name="base_length" value="0.14" /> <!-- Length - wysokosc podstawy -->
     <xacro:property name="wheel_radius" value="0.1" />
     <xacro:property name="wheel_length" value="0.05" />
@@ -22,5 +22,5 @@
             <origin xyz="0 0 ${base_length / 2.0}" rpy="0 0 0" />
         </collision>
-        <xacro:cylinder_inertia m="5.0" r="${base_diameter / 2.0}" h="${base_length}"
+        <xacro:cylinder_inertia m="5.0" r="${2*base_diameter / 2.0}" h="${2*base_length}"
                                 xyz="0 0 ${base_length / 2.0}" rpy="0 0 0" />
     </link>
@@ -74,5 +74,5 @@
                 <origin xyz="0 0 0" rpy="${pi / 2.0} 0 0" />
             </collision>
-            <xacro:cylinder_inertia m="1.0" r="${wheel_radius}" h="${wheel_length}"
+            <xacro:cylinder_inertia m="2.0" r="${2*wheel_radius}" h="${2*wheel_length}"
                                     xyz="0 0 0" rpy="${pi / 2.0} 0 0" />
         </link>
@@ -83,5 +83,5 @@
         <visual>
             <geometry>
-                <sphere radius="${(wheel_radius + 0.02) / 2.0}" />
+                <sphere radius="${(wheel_radius) / 2.0}" />
             </geometry>
             <origin xyz="0 0 0" rpy="0 0 0" />
@@ -94,5 +94,5 @@
             <origin xyz="0 0 0" rpy="0 0 0" />
         </collision>
-        <xacro:sphere_inertia m="5.0" r="${(wheel_radius + 0.02) / 2.0}"
+        <xacro:sphere_inertia m="8.0" r="${2*(wheel_radius + 0.02) / 2.0}"
                               xyz="0 0 0" rpy="0 0 0" />
     </link>
