Commit message: add lidar to robot

File: src/explorer_bot/urdf/common_properties.xacro (robot description, xacro)
@@ -9,4 +9,7 @@
     <material name="grey">
         <color rgba="0.5 0.5 0.5 1" />
+    </material>
+    <material name="red">
+        <color rgba="1 0 0 1" />
     </material>
     <xacro:macro name="cylinder_inertia" params="m r h xyz rpy">

File: src/explorer_bot/urdf/my_robot.urdf.xacro (robot description, xacro)
@@ -3,4 +3,5 @@
     <xacro:include filename="common_properties.xacro" />
     <xacro:include filename="mobile_base.xacro" />
+    <xacro:include filename="lidar.xacro" />
     <xacro:include filename="mobile_base_gazebo.xacro" />
 </robot>
